File: power.sch (EAGLE design)
At the start: 12 parts, among them IC1 7805T, J1 1X2-3.5MM

Commit message: Initial Commit
Connections:
- net N$3 renamed GND
Changed lines of the file:
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@@
 </variantdefs>
 <classes>
-<class number="0" name="default" width="0" drill="0">
+<class number="0" name="default" width="0.508" drill="30.48">
+<clearance class="0" value="1.016"/>
 </class>
 </classes>
@@
 </segment>
 </net>
-<net name="N$3" class="0">
+<net name="GND" class="0">
 <segment>
 <pinref part="D1" gate="1" pin="A"/>
@@
 <pinref part="JP1" gate="A" pin="2"/>
 <wire x1="99.06" y1="22.86" x2="106.68" y2="22.86" width="0.1524" layer="91"/>
+<label x="83.82" y="2.54" size="1.778" layer="95" xref="yes"/>
+<wire x1="83.82" y1="2.54" x2="81.28" y2="2.54" width="0.1524" layer="91"/>
+<wire x1="81.28" y1="2.54" x2="81.28" y2="10.16" width="0.1524" layer="91"/>
 </segment>
 </net>
